Commit message: Added gazebo model for jetbot

File: jetbot_mirea_description/urdf/common_properties.xacro (robot description, xacro)
@@ -20,4 +20,7 @@
     <material name="black">
         <color rgba="0.0 0.0 0.0 1" />
+    </material>
+    <material name="silver">
+        <color rgba="0.67 0.67 0.67 1.0" />
     </material>
     <!-- Specify some standard inertial calculations https://en.wikipedia.org/wiki/List_of_moments_of_inertia -->
