Commit message: Added new sensor: marvelmind (analog gps)

File: jetbot_mirea_description/urdf/gazebo_properties.xacro (robot description, xacro)
@@ -58,4 +58,11 @@
     </gazebo>
     <gazebo reference="back_camera_link">
+        <material>Gazebo/Red</material>
+        <mu1>0.2</mu1>
+        <mu2>0.2</mu2>
+        <kp>1000000.0</kp>
+        <kd>1.0</kd>
+    </gazebo>
+    <gazebo reference="marvelmind_link">
         <material>Gazebo/Red</material>
         <mu1>0.2</mu1>
@@ -225,3 +232,47 @@
         </sensor>
     </gazebo>
+    <!-- GPS (marvelmind)-->
+    <gazebo reference="marvelmind_link">
+        <sensor name="marvelmind_gps" type="gps">
+          <always_on>true</always_on>
+          <update_rate>30</update_rate>
+          <gps>
+            <position_sensing>
+              <horizontal>
+                <noise type="gaussian">
+                  <mean>0.0</mean>
+                  <stddev>2e-4</stddev>
+                </noise>
+              </horizontal>
+              <vertical>
+                <noise type="gaussian">
+                  <mean>0.0</mean>
+                  <stddev>2e-4</stddev>
+                </noise>
+              </vertical>
+            </position_sensing>
+            <velocity_sensing>
+              <horizontal>
+                <noise type="gaussian">
+                  <mean>0.0</mean>
+                  <stddev>2e-4</stddev>
+                </noise>
+              </horizontal>
+              <vertical>
+                <noise type="gaussian">
+                  <mean>0.0</mean>
+                  <stddev>2e-4</stddev>
+                </noise>
+              </vertical>
+            </velocity_sensing>
+          </gps>
+          <plugin name="marvelmind_gps_plugin" filename="libgazebo_ros_gps_sensor.so">
+            <ros>
+              <namespace>/gps</namespace>
+              <remapping>~/out:=data</remapping>
+              <remapping>~/vel:=velocity</remapping>
+            </ros>
+          </plugin>
+        </sensor>
+    </gazebo>
 </robot>

File: jetbot_mirea_description/urdf/jetbot_mirea_simple_gazebo_ideal.urdf.xacro (robot description, xacro)
@@ -30,4 +30,9 @@
     <xacro:property name="back_camera_height" value="0.02"/>
     <xacro:property name="back_camera_mass" value="0.05"/>
+    <!-- Параметры маяка marvelmind -->
+    <xacro:property name="marvelmind_lenght" value="0.04"/>
+    <xacro:property name="marvelmind_width" value="0.03"/>
+    <xacro:property name="marvelmind_height" value="0.015"/>
+    <xacro:property name="marvelmind_mass" value="0.05"/>
     <!-- "Импорты" модулей -->
     <xacro:include filename="$(find realsense_ros_gazebo)/xacro/depthcam.xacro"/>
@@ -116,4 +121,28 @@
         </xacro:inertial_box>
     </link>
+    <!-- Маяк marvelmind -->
+    <joint name="marvelmind_joint" type="fixed">
+        <parent link="computer_link"/>
+        <child link="marvelmind_link"/>
+        <origin xyz="0.0 0.0 ${computer_height/2 + marvelmind_height/2}" rpy="0 0 0"/>
+    </joint>
+    <link name="marvelmind_link">
+        <visual>
+            <origin xyz="0.0 0.0 0.0" rpy="0 0 0"/>
+            <geometry>
+                <box size="${marvelmind_lenght} ${marvelmind_width} ${marvelmind_height}"/>
+            </geometry>
+            <material name="orange"/>
+        </visual>
+        <collision>
+            <origin xyz="0.0 0.0 0.0" rpy="0 0 0"/>
+            <geometry>
+                <box size="${marvelmind_lenght} ${marvelmind_width} ${marvelmind_height}"/>
+            </geometry>
+        </collision>
+        <xacro:inertial_box mass="${marvelmind_mass}" x="${marvelmind_lenght}" y="${marvelmind_width}" z="${marvelmind_height}">
+            <origin xyz="0.0 0.0 0.0" rpy="0 0 0"/>
+        </xacro:inertial_box>
+    </link>
     <!-- Лидар -->
     <joint name="lidar_joint" type="fixed">

File: jetbot_mirea_description/urdf/jetbot_mirea_simple_gazebo_real.urdf.xacro (robot description, xacro)
@@ -30,4 +30,9 @@
     <xacro:property name="back_camera_height" value="0.02"/>
     <xacro:property name="back_camera_mass" value="0.05"/>
+    <!-- Параметры маяка marvelmind -->
+    <xacro:property name="marvelmind_lenght" value="0.04"/>
+    <xacro:property name="marvelmind_width" value="0.03"/>
+    <xacro:property name="marvelmind_height" value="0.015"/>
+    <xacro:property name="marvelmind_mass" value="0.05"/>
     <!-- "Импорты" модулей -->
     <xacro:include filename="$(find realsense_ros_gazebo)/xacro/depthcam.xacro"/>
@@ -140,4 +145,28 @@
         </xacro:inertial_cylinder>
     </link>
+    <!-- Маяк marvelmind -->
+    <joint name="marvelmind_joint" type="fixed">
+        <parent link="computer_link"/>
+        <child link="marvelmind_link"/>
+        <origin xyz="0.0 0.0 ${computer_height/2 + marvelmind_height/2}" rpy="0 0 0"/>
+    </joint>
+    <link name="marvelmind_link">
+        <visual>
+            <origin xyz="0.0 0.0 0.0" rpy="0 0 0"/>
+            <geometry>
+                <box size="${marvelmind_lenght} ${marvelmind_width} ${marvelmind_height}"/>
+            </geometry>
+            <material name="orange"/>
+        </visual>
+        <collision>
+            <origin xyz="0.0 0.0 0.0" rpy="0 0 0"/>
+            <geometry>
+                <box size="${marvelmind_lenght} ${marvelmind_width} ${marvelmind_height}"/>
+            </geometry>
+        </collision>
+        <xacro:inertial_box mass="${marvelmind_mass}" x="${marvelmind_lenght}" y="${marvelmind_width}" z="${marvelmind_height}">
+            <origin xyz="0.0 0.0 0.0" rpy="0 0 0"/>
+        </xacro:inertial_box>
+    </link>
     <!-- Основные приводные колеса -->
     <!-- Левое большое колесо -->
